File: v3.0/eagle/noisemaker_3-0.brd (EAGLE design)
At the start: 76.3 x 66.7 mm, 57 parts, among them IC1 REG1117, U3 ATMEGA32U4, Y1 16MHz

Commit message: board updates...
Parts:
- NPN: device transistor:TO220V -> SparkFun-DiscreteSemi:SOT23-3
- moved JP2 70.0 mm to (81.8, 20.3)
- moved JP3 38.1 mm to (71.1, 30.5), turned to 180 degrees
- moved R12 34.1 mm to (31.8, 35.6)
- moved R10 33.0 mm to (38.1, 36.8)
- moved AMP- 31.9 mm to (45.7, 2.54)
- moved AMP+ 31.4 mm to (40.6, 2.54)
- moved JP5 28.7 mm to (29.2, 6.35)
- moved R13 24.4 mm to (50.8, 35.6)
- moved NPN 24.3 mm to (53.3, 11.4)
- moved C9 22.2 mm to (40.6, 16.5)
- moved C11 21.6 mm to (40.6, 12.7)
- moved R8 16.7 mm to (62.2, 19.1)
- moved R11 13.3 mm to (58.4, 36.8)
- moved C8 12.8 mm to (59.7, 7.62)
- moved JP6 10.8 mm to (33.4, 1.78)
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Connections:
- net GND: now also NPN.2; no longer NPN.3
- net SPKR_OUT: now also NPN.3; no longer NPN.2

Commit message: updated board layout
Parts:
- moved JP1 60.5 mm to (90.9, 9.78)
- moved POLE2 53.3 mm to (58.4, 34.3)
- moved PH2 49.0 mm to (54.6, 24.1)
- moved R19 49.0 mm to (54.6, 20.3)
- moved LED2 48.7 mm to (57.1, 12.7)
- moved R7 47.0 mm to (63.5, 29.0), turned to 0 degrees
- moved R5 42.0 mm to (63.5, 26.5), turned to 0 degrees
- moved PH3 38.1 mm to (45.7, 24.1)
- moved R20 37.4 mm to (45.7, 20.3)
- moved R3 36.0 mm to (39.4, 7.62)
- moved LED7 35.3 mm to (30.5, 27.9)
- moved R13 34.9 mm to (16.5, 29.2)
- moved LED8 31.0 mm to (45.7, 27.9)
- moved R2 29.2 mm to (31.2, 7.75), turned to 270 degrees
- moved C2 29.0 mm to (5.59, 25.1), turned to 90 degrees
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Routing:
- net RAW: track 5.33 -> 0.00 mm

Commit message: updated board layout tues
Parts:
- added JP8: M01PTH_LONGPAD, SparkFun-Connectors:1X01_LONGPAD
- moved POLE3 10.2 mm to (2.54, 43.2)
Connections:
- net VCC: now also JP8.1
Routing:
- added copper zone on layer 1, net N$3
- added copper zone on layer 16, net N$3
Changed lines of the file:
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@@
 <layer number="27" name="tValues" color="7" fill="1" visible="no" active="yes"/>
 <layer number="28" name="bValues" color="7" fill="1" visible="no" active="yes"/>
-<layer number="29" name="tStop" color="7" fill="3" visible="no" active="yes"/>
-<layer number="30" name="bStop" color="7" fill="6" visible="no" active="yes"/>
+<layer number="29" name="tStop" color="7" fill="3" visible="yes" active="yes"/>
+<layer number="30" name="bStop" color="7" fill="6" visible="yes" active="yes"/>
 <layer number="31" name="tCream" color="7" fill="4" visible="no" active="yes"/>
 <layer number="32" name="bCream" color="7" fill="5" visible="no" active="yes"/>
@@
 <circle x="64.77" y="36.83" radius="1.016" width="0.254" layer="21"/>
 <circle x="5.461" y="2.159" radius="1.016" width="0.254" layer="21"/>
+<rectangle x1="-2.54" y1="40.64" x2="78.74" y2="67.31" layer="29"/>
+<rectangle x1="-3.81" y1="40.64" x2="77.47" y2="68.58" layer="30"/>
 </plain>
 <attributes>
@@
 <element name="R14" library="SparkFun-Passives" package="1206" value="" x="54.61" y="27.94"/>
 <element name="R18" library="SparkFun-Passives" package="1206" value="" x="38.1" y="27.94"/>
-<element name="POLE3" library="SparkFun-Connectors" package="1X01_LONGPAD" value="M01PTH_LONGPAD" x="7.62" y="34.29"/>
+<element name="POLE3" library="SparkFun-Connectors" package="1X01_LONGPAD" value="M01PTH_LONGPAD" x="2.54" y="43.18"/>
+<element name="JP8" library="SparkFun-Connectors" package="1X01_LONGPAD" value="M01PTH_LONGPAD" x="73.66" y="43.18"/>
 </elements>
 <signals>
@@
 <contactref element="R18" pad="2"/>
 <contactref element="U$1" pad="RING"/>
-<wire x1="67.9704" y1="20.0406" x2="71.12" y2="31.73" width="0" layer="19" extent="1-1"/>
-<wire x1="63.63" y1="16.51" x2="67.9704" y2="20.0406" width="0" layer="19" extent="1-1"/>
-<wire x1="60.83" y1="19.05" x2="63.63" y2="16.51" width="0" layer="19" extent="1-1"/>
-<wire x1="60.83" y1="21.59" x2="60.83" y2="19.05" width="0" layer="19" extent="1-1"/>
-<wire x1="57.15" y1="14.45" x2="60.83" y2="19.05" width="0" layer="19" extent="1-1"/>
-<wire x1="53.21" y1="20.32" x2="57.15" y2="14.45" width="0" layer="19" extent="1-1"/>
-<wire x1="57.79" y1="6.35" x2="57.15" y2="14.45" width="0" layer="19" extent="1-1"/>
-<wire x1="57.79" y1="2.54" x2="57.79" y2="6.35" width="0" layer="19" extent="1-1"/>
-<wire x1="51.12" y1="4.81" x2="57.79" y2="6.35" width="0" layer="19" extent="1-1"/>
-<wire x1="44.32" y1="20.32" x2="53.21" y2="20.32" width="0" layer="19" extent="1-1"/>
-<wire x1="35.43" y1="20.32" x2="44.32" y2="20.32" width="0" layer="19" extent="1-1"/>
-<wire x1="39.5" y1="27.94" x2="35.43" y2="20.32" width="0" layer="19" extent="1-1"/>
-<wire x1="38.1" y1="32.89" x2="39.5" y2="27.94" width="0" layer="19" extent="1-1"/>
-<wire x1="25.4" y1="26.67" x2="35.43" y2="20.32" width="0" layer="19" extent="1-1"/>
-<wire x1="17.91" y1="29.21" x2="25.4" y2="26.67" width="0" layer="19" extent="1-1"/>
-<wire x1="14.605" y1="24.296" x2="17.91" y2="29.21" width="0" layer="19" extent="1-1"/>
-<wire x1="12.27015" y1="19.2025875" x2="14.605" y2="24.296" width="0" layer="19" extent="1-1"/>
-<wire x1="10.29" y1="29.21" x2="14.605" y2="24.296" width="0" layer="19" extent="1-1"/>
-<wire x1="5.588" y1="25.996" x2="10.29" y2="29.21" width="0" layer="19" extent="1-1"/>
-<wire x1="1.27" y1="24.638" x2="5.588" y2="25.996" width="0" layer="19" extent="1-1"/>
-<wire x1="1.27" y1="22.098" x2="1.27" y2="24.638" width="0" layer="19" extent="1-1"/>
-<wire x1="8.310353125" y1="12.69720625" x2="12.27015" y2="19.2025875" width="0" layer="19" extent="1-1"/>
 <wire x1="6.1341" y1="5.854240625" x2="8.310353125" y2="12.69720625" width="0" layer="19" extent="1-1"/>
-<wire x1="19.906903125" y1="17.50553125" x2="12.27015" y2="19.2025875" width="0" layer="19" extent="1-1"/>
-<wire x1="21.603959375" y1="12.131521875" x2="19.906903125" y2="17.50553125" width="0" layer="19" extent="1-1"/>
-<wire x1="17.078475" y1="7.6060375" x2="21.603959375" y2="12.131521875" width="0" layer="19" extent="1-1"/>
-<wire x1="13.96720625" y1="7.040353125" x2="17.078475" y2="7.6060375" width="0" layer="19" extent="1-1"/>
-<wire x1="25.1739375" y1="6.19460625" x2="21.603959375" y2="12.131521875" width="0" layer="19" extent="1-1"/>
-<wire x1="28.3337" y1="6.235240625" x2="25.1739375" y2="6.19460625" width="0" layer="19" extent="1-1"/>
-<wire x1="33.401" y1="1.778" x2="28.3337" y2="6.235240625" width="0" layer="19" extent="1-1"/>
-<wire x1="54.61" y1="32.89" x2="53.21" y2="20.32" width="0" layer="19" extent="1-1"/>
-<wire x1="72.81" y1="4.98" x2="63.63" y2="16.51" width="0" layer="19" extent="1-1"/>
 </signal>
 <signal name="AREF">
@@
 <contactref element="MODE" pad="2"/>
 <contactref element="MODE" pad="1"/>
+<contactref element="JP8" pad="1"/>
+<wire x1="62.1" y1="31.623" x2="73.66" y2="43.18" width="0" layer="19" extent="1-1"/>
 <wire x1="58.42" y1="34.29" x2="62.1" y2="31.623" width="0" layer="19" extent="1-1"/>
 <wire x1="53.21" y1="27.94" x2="58.42" y2="34.29" width="0" layer="19" extent="1-1"/>
@@
 <contactref element="POLE3" pad="1"/>
 <contactref element="R12" pad="2"/>
-<wire x1="7.49" y1="29.21" x2="7.62" y2="34.29" width="0" layer="19" extent="1-1"/>
+<wire x1="7.49" y1="29.21" x2="2.54" y2="43.18" width="0" layer="19" extent="1-1"/>
 <wire x1="18.209846875" y1="8.737409375" x2="7.49" y2="29.21" width="0" layer="19" extent="1-1"/>
 <wire x1="20.701" y1="1.778" x2="18.209846875" y2="8.737409375" width="0" layer="19" extent="1-1"/>
@@
 <wire x1="44.45" y1="27.94" x2="56.01" y2="27.94" width="0" layer="19" extent="1-1"/>
 </signal>
+<signal name="N$3">
+<polygon width="0.4064" layer="1">
+<vertex x="-3.81" y="68.58"/>
+<vertex x="25.4" y="68.58"/>
+<vertex x="25.4" y="40.64"/>
+<vertex x="-3.81" y="40.64"/>
+</polygon>
+<polygon width="0.4064" layer="16">
+<vertex x="-5.08" y="69.85"/>
+<vertex x="27.94" y="69.85"/>
+<vertex x="27.94" y="40.64"/>
+<vertex x="-5.08" y="40.64"/>
+</polygon>
+<polygon width="0.4064" layer="1">
+<vertex x="50.8" y="68.58"/>
+<vertex x="80.01" y="68.58"/>
+<vertex x="80.01" y="40.64"/>
+<vertex x="50.8" y="40.64"/>
+</polygon>
+<polygon width="0.4064" layer="16">
+<vertex x="45.72" y="69.85"/>
+<vertex x="78.74" y="69.85"/>
+<vertex x="78.74" y="40.64"/>
+<vertex x="45.72" y="40.64"/>
+</polygon>
+</signal>
 </signals>

Commit message: merging in @shanqiu's latest updates
Parts:
- removed PH3: M9960_11B, photo-elements:M9960
- removed R20: (no value), SparkFun-Passives:1206
- added JP9, LED_STRIP: (no value), pinhead:1X03/90
Connections:
- new net N$11: LED_STRIP.3
- new net N$6: LED_STRIP.1
- net A4: now also JP9.2; no longer PH3.2, R20.2
- net D6: now also LED_STRIP.2
- net GND: now also JP9.3; no longer R20.1
- net VCC: now also JP9.1; no longer PH3.1
Changed lines of the file:
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@@
 <?xml version="1.0" encoding="utf-8"?>
 <!DOCTYPE eagle SYSTEM "eagle.dtd">
-<eagle version="6.4">
+<eagle version="6.5.0">
 <drawing>
 <settings>
@@
 <element name="R15" library="SparkFun-Passives" package="1206" value="" x="36.83" y="20.32"/>
 <element name="R19" library="SparkFun-Passives" package="1206" value="" x="54.61" y="20.32"/>
-<element name="R20" library="SparkFun-Passives" package="1206" value="" x="45.72" y="20.32"/>
 <element name="PH2" library="photo-elements" package="M9960" value="M9960_11B" x="54.61" y="24.13"/>
-<element name="PH3" library="photo-elements" package="M9960" value="M9960_11B" x="45.72" y="24.13"/>
 <element name="JP5" library="SparkFun" package="2X3" value="AVR_SPI" x="20.32" y="24.13"/>
 <element name="U$1" library="adafruit" package="PJ-102A" value="2.1MMJACKTHM" x="76.2" y="5.08" rot="R270"/>
@@
 <element name="POLE3" library="SparkFun-Connectors" package="1X01_LONGPAD" value="M01PTH_LONGPAD" x="2.54" y="43.18"/>
 <element name="JP8" library="SparkFun-Connectors" package="1X01_LONGPAD" value="M01PTH_LONGPAD" x="73.66" y="43.18"/>
+<element name="JP9" library="pinhead" package="1X03/90" value="" x="-12.7" y="5.08"/>
+<element name="LED_STRIP" library="pinhead" package="1X03/90" value="" x="-25.4" y="5.08"/>
 </elements>
 <signals>
@@
 <contactref element="NPN" pad="2"/>
 <contactref element="R8" pad="1"/>
-<contactref element="R20" pad="1"/>
 <contactref element="R19" pad="1"/>
 <contactref element="R15" pad="1"/>
@@
 <contactref element="R18" pad="2"/>
 <contactref element="U$1" pad="RING"/>
+<contactref element="JP9" pad="3"/>
+<wire x1="67.9704" y1="20.0406" x2="71.12" y2="31.73" width="0" layer="19" extent="1-1"/>
+<wire x1="63.63" y1="16.51" x2="67.9704" y2="20.0406" width="0" layer="19" extent="1-1"/>
+<wire x1="60.83" y1="19.05" x2="63.63" y2="16.51" width="0" layer="19" extent="1-1"/>
+<wire x1="60.83" y1="21.59" x2="60.83" y2="19.05" width="0" layer="19" extent="1-1"/>
+<wire x1="57.15" y1="14.45" x2="60.83" y2="19.05" width="0" layer="19" extent="1-1"/>
+<wire x1="53.21" y1="20.32" x2="57.15" y2="14.45" width="0" layer="19" extent="1-1"/>
+<wire x1="57.79" y1="6.35" x2="57.15" y2="14.45" width="0" layer="19" extent="1-1"/>
+<wire x1="57.79" y1="2.54" x2="57.79" y2="6.35" width="0" layer="19" extent="1-1"/>
+<wire x1="51.12" y1="4.81" x2="57.79" y2="6.35" width="0" layer="19" extent="1-1"/>
+<wire x1="54.61" y1="32.89" x2="53.21" y2="20.32" width="0" layer="19" extent="1-1"/>
+<wire x1="72.81" y1="4.98" x2="63.63" y2="16.51" width="0" layer="19" extent="1-1"/>
+<wire x1="39.5" y1="27.94" x2="53.21" y2="20.32" width="0" layer="19" extent="1-1"/>
+<wire x1="38.1" y1="32.89" x2="39.5" y2="27.94" width="0" layer="19" extent="1-1"/>
+<wire x1="35.43" y1="20.32" x2="39.5" y2="27.94" width="0" layer="19" extent="1-1"/>
+<wire x1="25.4" y1="26.67" x2="35.43" y2="20.32" width="0" layer="19" extent="1-1"/>
+<wire x1="17.91" y1="29.21" x2="25.4" y2="26.67" width="0" layer="19" extent="1-1"/>
+<wire x1="14.605" y1="24.296" x2="17.91" y2="29.21" width="0" layer="19" extent="1-1"/>
+<wire x1="12.27015" y1="19.2025875" x2="14.605" y2="24.296" width="0" layer="19" extent="1-1"/>
+<wire x1="10.29" y1="29.21" x2="14.605" y2="24.296" width="0" layer="19" extent="1-1"/>
+<wire x1="5.588" y1="25.996" x2="10.29" y2="29.21" width="0" layer="19" extent="1-1"/>
+<wire x1="1.27" y1="24.638" x2="5.588" y2="25.996" width="0" layer="19" extent="1-1"/>
+<wire x1="1.27" y1="22.098" x2="1.27" y2="24.638" width="0" layer="19" extent="1-1"/>
+<wire x1="8.310353125" y1="12.69720625" x2="12.27015" y2="19.2025875" width="0" layer="19" extent="1-1"/>
 <wire x1="6.1341" y1="5.854240625" x2="8.310353125" y2="12.69720625" width="0" layer="19" extent="1-1"/>
+<wire x1="19.906903125" y1="17.50553125" x2="12.27015" y2="19.2025875" width="0" layer="19" extent="1-1"/>
+<wire x1="21.603959375" y1="12.131521875" x2="19.906903125" y2="17.50553125" width="0" layer="19" extent="1-1"/>
+<wire x1="17.078475" y1="7.6060375" x2="21.603959375" y2="12.131521875" width="0" layer="19" extent="1-1"/>
+<wire x1="13.96720625" y1="7.040353125" x2="17.078475" y2="7.6060375" width="0" layer="19" extent="1-1"/>
+<wire x1="25.1739375" y1="6.19460625" x2="21.603959375" y2="12.131521875" width="0" layer="19" extent="1-1"/>
+<wire x1="28.3337" y1="6.235240625" x2="25.1739375" y2="6.19460625" width="0" layer="19" extent="1-1"/>
+<wire x1="33.401" y1="1.778" x2="28.3337" y2="6.235240625" width="0" layer="19" extent="1-1"/>
+<wire x1="-10.16" y1="1.27" x2="6.1341" y2="5.854240625" width="0" layer="19" extent="1-1"/>
 </signal>
 <signal name="AREF">
@@
 <contactref element="AMP+" pad="1"/>
 <contactref element="PH1" pad="1"/>
-<contactref element="PH3" pad="1"/>
 <contactref element="PH2" pad="1"/>
 <contactref element="JP5" pad="2"/>
@@
 <contactref element="MODE" pad="1"/>
 <contactref element="JP8" pad="1"/>
+<contactref element="JP9" pad="1"/>
 <wire x1="62.1" y1="31.623" x2="73.66" y2="43.18" width="0" layer="19" extent="1-1"/>
 <wire x1="58.42" y1="34.29" x2="62.1" y2="31.623" width="0" layer="19" extent="1-1"/>
 <wire x1="53.21" y1="27.94" x2="58.42" y2="34.29" width="0" layer="19" extent="1-1"/>
 <wire x1="52.86" y1="24.13" x2="53.21" y2="27.94" width="0" layer="19" extent="1-1"/>
-<wire x1="43.97" y1="24.13" x2="52.86" y2="24.13" width="0" layer="19" extent="1-1"/>
-<wire x1="35.08" y1="24.13" x2="43.97" y2="24.13" width="0" layer="19" extent="1-1"/>
-<wire x1="28.222" y1="21.336" x2="35.08" y2="24.13" width="0" layer="19" extent="1-1"/>
-<wire x1="28.349" y1="18.796" x2="28.222" y2="21.336" width="0" layer="19" extent="1-1"/>
-<wire x1="22.16964375" y1="12.69720625" x2="28.349" y2="18.796" width="0" layer="19" extent="1-1"/>
-<wire x1="16.512790625" y1="7.040353125" x2="22.16964375" y2="12.69720625" width="0" layer="19" extent="1-1"/>
-<wire x1="8.8760375" y1="12.131521875" x2="16.512790625" y2="7.040353125" width="0" layer="19" extent="1-1"/>
-<wire x1="12.835834375" y1="19.768275" x2="8.8760375" y2="12.131521875" width="0" layer="19" extent="1-1"/>
-<wire x1="20.32" y1="26.67" x2="28.222" y2="21.336" width="0" layer="19" extent="1-1"/>
 <wire x1="48.9712" y1="36.5506" x2="53.21" y2="27.94" width="0" layer="19" extent="1-1"/>
 <wire x1="42.4688" y1="36.5506" x2="48.9712" y2="36.5506" width="0" layer="19" extent="1-1"/>
@@
 <wire x1="67.9704" y1="17.7546" x2="63.63" y2="19.05" width="0" layer="19" extent="1-1"/>
 <wire x1="61.59" y1="6.35" x2="61.207" y2="10.922" width="0" layer="19" extent="1-1"/>
+<wire x1="20.32" y1="26.67" x2="27.2288" y2="36.5506" width="0" layer="19" extent="1-1"/>
+<wire x1="28.222" y1="21.336" x2="20.32" y2="26.67" width="0" layer="19" extent="1-1"/>
+<wire x1="28.349" y1="18.796" x2="28.222" y2="21.336" width="0" layer="19" extent="1-1"/>
+<wire x1="35.08" y1="24.13" x2="28.222" y2="21.336" width="0" layer="19" extent="1-1"/>
+<wire x1="22.16964375" y1="12.69720625" x2="28.349" y2="18.796" width="0" layer="19" extent="1-1"/>
+<wire x1="16.512790625" y1="7.040353125" x2="22.16964375" y2="12.69720625" width="0" layer="19" extent="1-1"/>
+<wire x1="8.8760375" y1="12.131521875" x2="16.512790625" y2="7.040353125" width="0" layer="19" extent="1-1"/>
+<wire x1="12.835834375" y1="19.768275" x2="8.8760375" y2="12.131521875" width="0" layer="19" extent="1-1"/>
 <wire x1="31.242" y1="6.347" x2="22.16964375" y2="12.69720625" width="0" layer="19" extent="1-1"/>
 <wire x1="28.321" y1="1.778" x2="31.242" y2="6.347" width="0" layer="19" extent="1-1"/>
@@
 <wire x1="40.77" y1="7.62" x2="39.37" y2="2.54" width="0" layer="19" extent="1-1"/>
 <wire x1="45.59" y1="7.62" x2="40.77" y2="7.62" width="0" layer="19" extent="1-1"/>
+<wire x1="-15.24" y1="1.27" x2="8.8760375" y2="12.131521875" width="0" layer="19" extent="1-1"/>
 </signal>
 <signal name="RAW" class="1">
@@
 <signal name="A4">
 <contactref element="U3" pad="40"/>
-<contactref element="R20" pad="2"/>
-<contactref element="PH3" pad="2"/>
-<wire x1="47.12" y1="20.32" x2="47.47" y2="24.13" width="0" layer="19" extent="1-1"/>
-<wire x1="19.906903125" y1="10.434465625" x2="47.12" y2="20.32" width="0" layer="19" extent="1-1"/>
+<contactref element="JP9" pad="2"/>
+<wire x1="-12.7" y1="1.27" x2="19.906903125" y2="10.434465625" width="0" layer="19" extent="1-1"/>
 </signal>
 <signal name="A3">
@@
 <contactref element="JP7" pad="4"/>
 <contactref element="U3" pad="27"/>
-<wire x1="1.27" y1="9.398" x2="10.57309375" y2="10.434465625" width="0" layer="19" extent="1-1"/>
+<contactref element="LED_STRIP" pad="2"/>
+<wire x1="1.27" y1="9.398" x2="-25.4" y2="1.27" width="0" layer="19" extent="1-1"/>
+<wire x1="10.57309375" y1="10.434465625" x2="1.27" y2="9.398" width="0" layer="19" extent="1-1"/>
 </signal>
 <signal name="D7">
@@
 </polygon>
 </signal>
+<signal name="N$6">
+<contactref element="LED_STRIP" pad="1"/>
+</signal>
+<signal name="N$11">
+<contactref element="LED_STRIP" pad="3"/>
+</signal>
 </signals>
