File: v4.0/eagle/noisemaker_4-0.brd (EAGLE design)
At the start: 81.3 x 68.5 mm, 61 parts, among them U1 MIC5219 5V

Commit message: 4.0 completed with gerber exports
Parts:
- removed C11: 0.1uF, SparkFun-Capacitors:1206
- removed F2: 500mA, SparkFun:PTC-1206
- removed JP3: USB-B, SparkFun-Connectors:USB-B-PTH
- removed LED2: (no value), adafruit:LED3MM
- removed LED3: (no value), adafruit:1206
- removed Q1: (no value), SparkFun-DiscreteSemi:TO-92-AMMO
- removed R15, R19: 10k, SparkFun-Passives:1206
- removed R18: 330, SparkFun-Passives:1206
- removed RANGE: (no value), switch-omron:B3F-10XX
- removed RV1: (no value), SparkFun-Electromechanical:ALPS_POT
- removed TP1: TEST-POINTTP_15TH_THRU, SparkFun-Passives:TP_15TH
- removed U$1: 2.1MMJACKTHM, adafruit:PJ-102A
- removed U1: MIC5219 5V, SparkFun-PowerIC:SOT23-5
- added C3: 0.1uF, SparkFun-Capacitors:1206
- added F1: 500mA, SparkFun:PTC-1206
- added JP5: JUMPER-PAD-2-NC_BY_TRACENO_SILK, SparkFun-Passives:PAD-JUMPER-2-NC_BY_TRACE_NO_SILK
- added PWRJACK: 2.1MMJACKTHM, adafruit:PJ-102A
- added USB: USB-CON-5PIN-105017-0001, GeekAmmo:USB-MICRO-MOLEX-105017-0001
- added VOL: (no value), SparkFun-Electromechanical:ALPS_POT
- added VREG: MIC5219 5V, SparkFun-PowerIC:SOT23-5
- LED1: value (none) -> WS2812B3535; device adafruit:LED3MM -> adafruit:LED3535
- POLE1, POLE2: value M01PTH_LONGPAD -> (none); device SparkFun-Connectors:1X01_LONGPAD -> SparkFun-Connectors:1X01_ALLIGATOR_3MM
- R11: value 10k -> 1k
- R13: value 1k -> 10k
- R14: value 330 -> 10k
- R4: value 330 -> 22
- R7: value 22 -> 330
- moved POLE2 51.1 mm to (11.4, 47.0), turned to 90 degrees
- moved R13 46.5 mm to (58.7, 33.1), turned to 180 degrees
- moved R11 43.8 mm to (10.9, 35.6), turned to 270 degrees
- moved POLE1 40.2 mm to (57.1, 47.0), turned to 90 degrees
- moved R7 32.9 mm to (29.3, 24.0), turned to 270 degrees
- moved R8 28.4 mm to (34.3, 8.89), turned to 90 degrees
- moved SENSOR1 27.2 mm to (65.0, 35.9)
- moved R4 26.9 mm to (56.5, 27.9), turned to 0 degrees
- moved JP2 21.4 mm to (67.1, 10.9)
- moved SENSOR2 19.4 mm to (58.8, 35.9)
- moved R2 16.4 mm to (13.6, 35.6)
- moved R10 12.8 mm to (26.4, 24.0), turned to 90 degrees
- moved R14 11.1 mm to (65.0, 33.0), turned to 180 degrees
- moved LED1 10.5 mm to (34.3, 16.5), turned to 0 degrees
- moved TX 9.08 mm to (32.0, 24.0)
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Connections:
- removed net N$12: LED1.K, R18.1
- removed net N$13: LED2.A, R14.2
- removed net N$8: JP3.D+, R5.2
- removed net N$9: JP3.D-, R7.2
- new net 3.3V: LED1.2
- new net N$11: R4.2, USB.3
- new net N$14: R5.2, USB.2
- net A0: now also POLE2.1@0, POLE2.1@2, R11.1; no longer POLE1.1, R13.1
- net A2: now also R14.2; no longer R15.2
- net A3: now also R13.2; no longer R19.2
- net D+: now also R4.1; no longer R5.1
- net D-: now also R5.1; no longer R7.1
- net D14: now also R7.1; no longer R4.1
- net D5: now also LED1.1; no longer LED1.A, LED2.K
- net D7: no longer R11.2, RANGE.3, RANGE.4
- net D8: no longer Q1.2
- net GND: now also C3.1, JP5.1, LED1.4, PWRJACK.RING, R11.2, R13.1, R14.1, USB.5, VREG.2; no longer C11.1, JP3.GND, Q1.1, R11.1, R13.2, R15.1, R18.2, R19.1, U$1.RING, U1.2
- net N$3: now also VOL.P$1; no longer RV1.P$1
- net N$5: now also R7.2; no longer R4.2
- net N$6: now also JP5.2, VOL.P$3; no longer RV1.P$3, TP1.P$1
- net RAW: now also PWRJACK.TIP, VREG.1, VREG.3; no longer U$1.TIP, U1.1, U1.3
- net SPKR_OUT: now also VOL.P$2; no longer Q1.3, RV1.P$2
- net UVCC: now also F1.1, USB.1; no longer F2.1, JP3.VBUS
- net VCC: now also C3.2, F1.2, POLE1.1@0, POLE1.1@2, VREG.5; no longer C11.2, F2.2, POLE2.1, R14.1, RANGE.1, RANGE.2, U1.5
Routing:
- net VCC: track 0.00 -> 261.1 mm, vias 0 -> 3
- net UVCC: track 0.00 -> 84.7 mm, vias 0 -> 4
- net D8: track 0.00 -> 72.8 mm, vias 0 -> 3
- net A2: track 0.00 -> 61.7 mm, vias 0 -> 2
- net A3: track 0.00 -> 58.7 mm
- net A0: track 0.00 -> 54.0 mm, vias 0 -> 2
- net A1: track 0.00 -> 41.1 mm, vias 0 -> 1
- net D+: track 0.00 -> 39.2 mm, vias 0 -> 2
- net D-: track 0.00 -> 37.4 mm
- net D2: track 0.00 -> 35.5 mm, vias 0 -> 2
- net N$3: track 0.00 -> 30.2 mm
- net N$4: track 0.00 -> 28.8 mm
- net RAW: track 0.00 -> 27.6 mm
- net SPKR_OUT: track 0.00 -> 25.9 mm
- net D11: track 0.00 -> 25.1 mm, vias 0 -> 1
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Other:
- board size 81.3 x 68.5 mm -> 68.6 x 68.5 mm
- board text added: "Parsons Design + Technology"
- board text added: "VOL"
- board text added: "jos.ph 2017"
- board text added: "v4"
- board text removed: "L.Campbell J.Brucker-Cohen K.Moriwaki J.McDonald T.Gou N.Messier T.Wen J.Saavedra"
- board text removed: "gadgIteration"
- board text removed: "gadgiteration.org"
- board text removed: "special thanks: Sven // Vivian // Ben May 2014"
- board text removed: "v3.0"
