File: v4.0/eagle/noisemaker_4-0.sch (EAGLE design)
At the start: 61 parts, among them U1 MIC5219 5V

Commit message: 4.0 completed with gerber exports
Parts:
- removed JP3: USB-B, SparkFun-Connectors:USBPTH
- removed LED2: (no value), adafruit:LED3MM
- removed LED3: (no value), adafruit:LEDSMT1206
- removed Q1: (no value), SparkFun-DiscreteSemi:TRANSISTOR_NPNTO-92-AMMO
- removed R15, R19: 10k, SparkFun-Passives:RESISTOR1206
- removed R18: 330, SparkFun-Passives:RESISTOR1206
- removed RANGE: (no value), switch-omron:10-XX
- removed TP1: TEST-POINTTP_15TH_THRU, SparkFun-Passives:TEST-POINTTP_15TH_THRU
- added JP5: JUMPER-PAD-2-NC_BY_TRACENO_SILK, SparkFun-Passives:JUMPER-PAD-2-NC_BY_TRACENO_SILK
- added USB: USB-CON-5PIN-105017-0001, GeekAmmo:USB-CON-5PIN-105017-0001
- LED1: value (none) -> WS2812B3535; device adafruit:LED3MM -> adafruit:WS2812B3535
- POLE1, POLE2: value M01PTH_LONGPAD -> M01ALLIGATOR-3MM; device SparkFun-Connectors:M01PTH_LONGPAD -> SparkFun-Connectors:M01ALLIGATOR-3MM
- R11: value 10k -> 1k
- R13: value 1k -> 10k
- R14: value 330 -> 10k
- R4: value 330 -> 22
- R7: value 22 -> 330
- renumbered C11 to C3, F2 to F1, RV1 to VOL, U$1 to PWRJACK, U1 to VREG
Connections:
- removed net N$12: LED1.C, R18.1
- removed net N$13: LED2.A, R14.2
- removed net N$8: JP3.D+, R5.2
- removed net N$9: JP3.D-, R7.2
- new net 3.3V: LED1.VDD
- new net N$11: R4.2, USB.D+
- new net N$14: R5.2, USB.D-
- net A0: now also POLE2.1, R11.1; no longer POLE1.1, R13.1
- net A2: now also R14.2; no longer R15.2
- net A3: now also R13.2; no longer R19.2
- net D+: now also R4.1; no longer R5.1
- net D-: now also R5.1; no longer R7.1
- net D14: now also R7.1; no longer R4.1
- net D5: now also LED1.DI; no longer LED1.A, LED2.C
- net D7: no longer R11.2, RANGE.P, RANGE.P1
- net D8: no longer Q1.B
- net GND: now also JP5.1, LED1.GND, R11.2, R13.1, R14.1, USB.GND; no longer JP3.GND, Q1.E, R11.1, R13.2, R15.1, R18.2, R19.1
- net N$5: now also R7.2; no longer R4.2
- net N$6: now also JP5.2; no longer TP1.1
- net SPKR_OUT: no longer Q1.C
- net UVCC: now also USB.VBUS; no longer JP3.VBUS
- net VCC: now also POLE1.1; no longer POLE2.1, R14.1, RANGE.S, RANGE.S1
Other:
- note added: "indicator LED"
- note removed: "Human vs Normal Indicator LEDs"
- moved on the sheet: MODE, POLE1, POLE2, R10, R11, R13, R14, R4, R5, R7
